File: USB-ISO-RS485/USB-ISO-RS485.sch (KiCad schematic (older format))
At the start: 39 parts, among them P1 WAGO 233-503, P10 TST, P11 TST, P12 TST, P2 USB_A, P9 TST, U1 ADM2582E, U2 FT232RL

Commit message: new PDF export
Parts:
- D3, D4, D5: value TVS -> P6SMB 6,8CA
- gave numbers to parts that had none: 5
Changed lines of the file:
@@
 U 1 1 590F1246
 P 8200 5400
-F 0 "P2" H 8400 5200 50  0000 C CNN
+F 0 "P2" V 7900 5400 50  0000 C CNN
 F 1 "USB_A" H 8150 5600 50  0000 C CNN
 F 2 "Connectors:USB_B" V 8150 5300 60  0001 C CNN
@@
 $EndComp
 $Comp
-L GND #PWR18
+L GND #PWR01
 U 1 1 590F26A8
 P 6850 3700
-F 0 "#PWR18" H 6850 3450 50  0001 C CNN
+F 0 "#PWR01" H 6850 3450 50  0001 C CNN
 F 1 "GND" H 6850 3550 50  0000 C CNN
 F 2 "" H 6850 3700 60  0000 C CNN
@@
 $EndComp
 $Comp
-L GND #PWR19
+L GND #PWR02
 U 1 1 590F2B53
 P 9500 5950
-F 0 "#PWR19" H 9500 5700 50  0001 C CNN
+F 0 "#PWR02" H 9500 5700 50  0001 C CNN
 F 1 "GND" H 9500 5800 50  0000 C CNN
 F 2 "" H 9500 5950 60  0000 C CNN
@@
 NoConn ~ 6850 2950
 $Comp
-L +5V #PWR14
+L +5V #PWR03
 U 1 1 590F2BAB
 P 6450 1250
-F 0 "#PWR14" H 6450 1100 50  0001 C CNN
+F 0 "#PWR03" H 6450 1100 50  0001 C CNN
 F 1 "+5V" H 6450 1390 50  0000 C CNN
 F 2 "" H 6450 1250 60  0000 C CNN
@@
 Connection ~ 6450 1400
 $Comp
-L +5V #PWR15
+L +5V #PWR04
 U 1 1 590F2C02
 P 6850 5550
-F 0 "#PWR15" H 6850 5400 50  0001 C CNN
+F 0 "#PWR04" H 6850 5400 50  0001 C CNN
 F 1 "+5V" H 6850 5690 50  0000 C CNN
 F 2 "" H 6850 5550 60  0000 C CNN
@@
 $EndComp
 $Comp
-L GND #PWR16
+L GND #PWR05
 U 1 1 590F2C1F
 P 6850 6000
-F 0 "#PWR16" H 6850 5750 50  0001 C CNN
+F 0 "#PWR05" H 6850 5750 50  0001 C CNN
 F 1 "GND" H 6850 5850 50  0000 C CNN
 F 2 "" H 6850 6000 60  0000 C CNN
@@
 $EndComp
 $Comp
-L +5V #PWR20
+L +5V #PWR06
 U 1 1 590F362B
 P 9350 2150
-F 0 "#PWR20" H 9350 2000 50  0001 C CNN
+F 0 "#PWR06" H 9350 2000 50  0001 C CNN
 F 1 "+5V" H 9350 2290 50  0000 C CNN
 F 2 "" H 9350 2150 60  0000 C CNN
@@
 	2000 2950 2050 2950
 $Comp
-L GND #PWR1
+L GND #PWR07
 U 1 1 590F46EB
 P 1250 2450
-F 0 "#PWR1" H 1250 2200 50  0001 C CNN
+F 0 "#PWR07" H 1250 2200 50  0001 C CNN
 F 1 "GND" H 1250 2300 50  0000 C CNN
 F 2 "" H 1250 2450 60  0000 C CNN
@@
 $EndComp
 $Comp
-L +3V3 #PWR10
+L +3V3 #PWR08
 U 1 1 590F640A
 P 4400 1700
-F 0 "#PWR10" H 4400 1550 50  0001 C CNN
+F 0 "#PWR08" H 4400 1550 50  0001 C CNN
 F 1 "+3V3" H 4400 1840 50  0000 C CNN
 F 2 "" H 4400 1700 60  0000 C CNN
@@
 $EndComp
 $Comp
-L GNDA #PWR11
+L GNDA #PWR09
 U 1 1 590F6460
 P 4500 2450
-F 0 "#PWR11" H 4500 2200 50  0001 C CNN
+F 0 "#PWR09" H 4500 2200 50  0001 C CNN
 F 1 "GNDA" H 4500 2300 50  0000 C CNN
 F 2 "" H 4500 2450 60  0000 C CNN
@@
 Connection ~ 4150 1800
 $Comp
-L GND #PWR3
+L GND #PWR010
 U 1 1 590F6C16
 P 2550 3850
-F 0 "#PWR3" H 2550 3600 50  0001 C CNN
+F 0 "#PWR010" H 2550 3600 50  0001 C CNN
 F 1 "GND" H 2550 3700 50  0000 C CNN
 F 2 "" H 2550 3850 60  0000 C CNN
@@
 Connection ~ 2550 3700
 $Comp
-L GNDA #PWR4
+L GNDA #PWR011
 U 1 1 590F6D6A
 P 3200 3850
-F 0 "#PWR4" H 3200 3600 50  0001 C CNN
+F 0 "#PWR011" H 3200 3600 50  0001 C CNN
 F 1 "GNDA" H 3200 3700 50  0000 C CNN
 F 2 "" H 3200 3850 60  0000 C CNN
@@
 $EndComp
 $Comp
-L GNDA #PWR7
+L GNDA #PWR012
 U 1 1 590F9E21
 P 3850 5550
-F 0 "#PWR7" H 3850 5300 50  0001 C CNN
+F 0 "#PWR012" H 3850 5300 50  0001 C CNN
 F 1 "GNDA" H 3850 5400 50  0000 C CNN
 F 2 "" H 3850 5550 60  0000 C CNN
@@
 	2400 5100 2300 5100
 $Comp
-L GND #PWR13
+L GND #PWR013
 U 1 1 590FB585
 P 6300 1650
-F 0 "#PWR13" H 6300 1400 50  0001 C CNN
+F 0 "#PWR013" H 6300 1400 50  0001 C CNN
 F 1 "GND" H 6300 1500 50  0000 C CNN
 F 2 "" H 6300 1650 60  0000 C CNN
@@
 	6350 2250 6850 2250
 $Comp
-L +5V #PWR22
+L +5V #PWR014
 U 1 1 590FBC4B
 P 10500 4950
-F 0 "#PWR22" H 10500 4800 50  0001 C CNN
+F 0 "#PWR014" H 10500 4800 50  0001 C CNN
 F 1 "+5V" H 10500 5090 50  0000 C CNN
 F 2 "" H 10500 4950 60  0000 C CNN
@@
 Connection ~ 6850 5600
 $Comp
-L GNDA #PWR5
+L GNDA #PWR015
 U 1 1 590FDE9F
 P 1200 6950
-F 0 "#PWR5" H 1200 6700 50  0001 C CNN
+F 0 "#PWR015" H 1200 6700 50  0001 C CNN
 F 1 "GNDA" H 1200 6800 50  0000 C CNN
 F 2 "" H 1200 6950 60  0000 C CNN
@@
 $EndComp
 $Comp
-L +3V3 #PWR8
+L +3V3 #PWR016
 U 1 1 590FDF0D
 P 1900 7050
-F 0 "#PWR8" H 1900 6900 50  0001 C CNN
+F 0 "#PWR016" H 1900 6900 50  0001 C CNN
 F 1 "+3V3" H 1900 7190 50  0000 C CNN
 F 2 "" H 1900 7050 60  0000 C CNN
@@
 $EndComp
 $Comp
-L +5V #PWR9
+L +5V #PWR017
 U 1 1 590FE4BA
 P 1900 7350
-F 0 "#PWR9" H 1900 7200 50  0001 C CNN
+F 0 "#PWR017" H 1900 7200 50  0001 C CNN
 F 1 "+5V" H 1900 7490 50  0000 C CNN
 F 2 "" H 1900 7350 60  0000 C CNN
@@
 $EndComp
 $Comp
-L GND #PWR6
+L GND #PWR018
 U 1 1 590FE52E
 P 1200 7250
-F 0 "#PWR6" H 1200 7000 50  0001 C CNN
+F 0 "#PWR018" H 1200 7000 50  0001 C CNN
 F 1 "GND" H 1200 7100 50  0000 C CNN
 F 2 "" H 1200 7250 60  0000 C CNN
@@
 	5800 4100 11100 4100
 $Comp
-L GNDA #PWR12
+L GNDA #PWR019
 U 1 1 59175054
 P 6400 4850
-F 0 "#PWR12" H 6400 4600 50  0001 C CNN
+F 0 "#PWR019" H 6400 4600 50  0001 C CNN
 F 1 "GNDA" H 6400 4700 50  0000 C CNN
 F 2 "" H 6400 4850 60  0000 C CNN
@@
 $EndComp
 $Comp
-L GND #PWR17
+L GND #PWR020
 U 1 1 591750CB
 P 6900 4850
-F 0 "#PWR17" H 6900 4600 50  0001 C CNN
+F 0 "#PWR020" H 6900 4600 50  0001 C CNN
 F 1 "GND" H 6900 4700 50  0000 C CNN
 F 2 "" H 6900 4850 60  0000 C CNN
@@
 P 8750 5300
 F 0 "D3" H 8500 5350 50  0000 C CNN
-F 1 "TVS" H 8500 5250 50  0000 C CNN
+F 1 "P6SMB 6,8CA" H 8550 5200 50  0000 C CNN
 F 2 "" H 8750 5300 60  0000 C CNN
 F 3 "" H 8750 5300 60  0000 C CNN
@@
 P 9150 5200
 F 0 "D4" H 8900 5250 50  0000 C CNN
-F 1 "TVS" H 8900 5150 50  0000 C CNN
+F 1 "P6SMB 6,8CA" H 9050 5100 50  0000 C CNN
 F 2 "" H 9150 5200 60  0000 C CNN
 F 3 "" H 9150 5200 60  0000 C CNN
@@
 P 9500 5100
 F 0 "D5" H 9250 5150 50  0000 C CNN
-F 1 "TVS" H 9250 5050 50  0000 C CNN
+F 1 "P6SMB 6,8CA" H 9500 5000 50  0000 C CNN
 F 2 "" H 9500 5100 60  0000 C CNN
 F 3 "" H 9500 5100 60  0000 C CNN
@@
 U 1 1 5946EA73
 P 8500 4950
-F 0 "R5" V 8580 4950 50  0000 C CNN
+F 0 "R5" V 8400 4950 50  0000 C CNN
 F 1 "0" V 8500 4950 50  0000 C CNN
 F 2 "" V 8430 4950 30  0000 C CNN
@@
 	9000 2200 9850 2200
 $Comp
-L R R?
+L R R4
 U 1 1 5946F4D2
 P 9250 3150
-F 0 "R?" V 9330 3150 50  0000 C CNN
+F 0 "R4" V 9330 3150 50  0000 C CNN
 F 1 "4k7" V 9250 3150 50  0000 C CNN
 F 2 "Resistors_SMD:R_0805_HandSoldering" V 9180 3150 30  0001 C CNN
@@
 $EndComp
 $Comp
-L R R?
+L R R6
 U 1 1 5946F6FB
 P 9700 2400
-F 0 "R?" V 9780 2400 50  0000 C CNN
+F 0 "R6" V 9780 2400 50  0000 C CNN
 F 1 "100k" V 9700 2400 50  0000 C CNN
 F 2 "Resistors_SMD:R_0805_HandSoldering" V 9630 2400 30  0001 C CNN
@@
 	9700 3150 9400 3150
 $Comp
-L IRF9540N Q?
+L IRF9540N Q1
 U 1 1 5946C4F1
 P 10050 2300
-F 0 "Q?" V 10300 2150 50  0000 L CNN
+F 0 "Q1" V 10300 2150 50  0000 L CNN
 F 1 "IRML6402" V 10400 2150 50  0000 L CNN
 F 2 "" H 10300 2225 50  0000 L CIN
@@
 	10250 2200 10350 2200
 $Comp
-L C_Small C?
+L C_Small C16
 U 1 1 5946D196
 P 10300 2550
-F 0 "C?" H 10310 2620 50  0000 L CNN
+F 0 "C16" H 10310 2620 50  0000 L CNN
 F 1 "100nF" H 10310 2470 50  0000 L CNN
 F 2 "Capacitors_SMD:C_0805_HandSoldering" H 10300 2550 60  0001 C CNN
@@
 	8450 2850 9000 2850
 $Comp
-L TST P?
+L TST P3
 U 1 1 5946EB1F
 P 3250 7350
-F 0 "P?" H 3250 7650 50  0000 C BNN
+F 0 "P3" H 3250 7650 50  0000 C BNN
 F 1 "TST" H 3250 7600 50  0000 C CNN
 F 2 "Measurement_Points:Measurement_Point_Round-TH_Small" H 3250 7350 60  0001 C CNN

Commit message: created new footprints & completed association.
Parts:
- D3, D4, D5: footprint (none) -> ADM2582E:P6SMB6,8CA
- FB1, R5: footprint (none) -> Resistors_SMD:R_0805_HandSoldering
- P1: footprint Connectors_WAGO:WAGO_734_3pin_Straight_RuggedPads -> ADM2582E:WAGO233-503
- Q1: value IRML6402 -> IRLML6402; footprint (none) -> ADM2582E:IRLML6402
Changed lines of the file:
@@
 F 0 "P1" H 4150 5500 50  0000 C CNN
 F 1 "WAGO 233-503" H 4250 5100 50  0000 C CNN
-F 2 "Connectors_WAGO:WAGO_734_3pin_Straight_RuggedPads" H 4150 5300 60  0001 C CNN
+F 2 "ADM2582E:WAGO233-503" H 4150 5300 60  0001 C CNN
 F 3 "" H 4150 5300 60  0000 C CNN
 	1    4150 5300
@@
 F 0 "FB1" H 9650 5750 50  0000 C CNN
 F 1 "BLM21PG 600" H 9550 5500 50  0000 C CNN
-F 2 "" H 9550 5600 60  0000 C CNN
+F 2 "Resistors_SMD:R_0805_HandSoldering" H 9550 5600 60  0001 C CNN
 F 3 "" H 9550 5600 60  0000 C CNN
 	1    9550 5600
@@
 F 0 "D3" H 8500 5350 50  0000 C CNN
 F 1 "P6SMB 6,8CA" H 8550 5200 50  0000 C CNN
-F 2 "" H 8750 5300 60  0000 C CNN
+F 2 "ADM2582E:P6SMB6,8CA" H 8750 5300 60  0001 C CNN
 F 3 "" H 8750 5300 60  0000 C CNN
 	1    8750 5300
@@
 F 0 "D4" H 8900 5250 50  0000 C CNN
 F 1 "P6SMB 6,8CA" H 9050 5100 50  0000 C CNN
-F 2 "" H 9150 5200 60  0000 C CNN
+F 2 "ADM2582E:P6SMB6,8CA" H 9150 5200 60  0001 C CNN
 F 3 "" H 9150 5200 60  0000 C CNN
 	1    9150 5200
@@
 F 0 "D5" H 9250 5150 50  0000 C CNN
 F 1 "P6SMB 6,8CA" H 9500 5000 50  0000 C CNN
-F 2 "" H 9500 5100 60  0000 C CNN
+F 2 "ADM2582E:P6SMB6,8CA" H 9500 5100 60  0001 C CNN
 F 3 "" H 9500 5100 60  0000 C CNN
 	1    9500 5100
@@
 F 0 "R5" V 8400 4950 50  0000 C CNN
 F 1 "0" V 8500 4950 50  0000 C CNN
-F 2 "" V 8430 4950 30  0000 C CNN
+F 2 "Resistors_SMD:R_0805_HandSoldering" V 8430 4950 30  0001 C CNN
 F 3 "" H 8500 4950 30  0000 C CNN
 	1    8500 4950
@@
 P 10050 2300
 F 0 "Q1" V 10300 2150 50  0000 L CNN
-F 1 "IRML6402" V 10400 2150 50  0000 L CNN
-F 2 "" H 10300 2225 50  0000 L CIN
+F 1 "IRLML6402" V 10400 2150 50  0000 L CNN
+F 2 "ADM2582E:IRLML6402" H 10300 2225 50  0001 L CIN
 F 3 "" H 10050 2300 50  0000 L CNN
 	1    10050 2300
